File: daisy.brd (EAGLE design)
At the start: 98.9 x 24.1 mm, 25 parts, among them IC1 ATMEGA, IC2 MCP1702-33, IC3 AT24CP, IC4 DS1307, Q1 32.768, U1 RJ45, X1 16 MHz, X3 JSTPH

Commit message: update
Parts:
- moved IC2 1.27 mm to (8.89, 11.7)
- moved C5 0.51 mm to (12.4, 20.6)
- moved R1 0.51 mm to (13.3, 13.8)
- moved J2 0.25 mm to (2.03, 9.14)
- moved X3 0.25 mm to (8.89, 4.32)
Routing:
- net D8: track 17.7 -> 32.6 mm, vias 1 -> 0
- net D7: track 30.6 -> 19.2 mm, vias 0 -> 1
- net VCC: track 112.4 -> 122.6 mm
- net GND: track 167.1 -> 173.9 mm, vias 0 -> 1
- net D10_SS: track 15.6 -> 20.5 mm, vias 1 -> 0
- net D6: track 17.7 -> 21.4 mm, vias 1 -> 2
- net A4_SDA: track 60.5 -> 57.2 mm, vias 0 -> 1
- net PWR: track 49.4 -> 52.0 mm
- net D9: track 27.2 -> 29.7 mm, vias 1 -> 0
- net D1_TX: track 39.8 -> 42.0 mm
- net A2: track 31.2 -> 32.6 mm
- net D13_SCK: track 18.7 -> 20.1 mm
- net N$1: track 12.7 -> 11.9 mm
- net N$21: track 12.2 -> 11.5 mm
Other:
- outline, holes or cut-outs redrawn
- board text added: "http://pvos.org/daisy"
- board text removed: "http://pvos.org/mowgli"
