File: daisy.sch (EAGLE design)
At the start: 25 parts, among them IC1 ATMEGA, IC2 MCP1702-33, IC3 AT24CP, IC4 DS1307, Q1 32.768, U1 RJ45, X1 16 MHz, X3 JSTPH

Commit message: update
Changed lines of the file:
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@@
 <pinref part="U$13" gate="G$1" pin="GND"/>
 <wire x1="182.88" y1="27.94" x2="187.96" y2="27.94" width="0.1524" layer="91"/>
+<junction x="182.88" y="17.78"/>
+<junction x="182.88" y="22.86"/>
+<junction x="182.88" y="25.4"/>
+<junction x="182.88" y="27.94"/>
 </segment>
 <segment>
